File: GardenLightingSystem/GardenLightingSystem.sch (KiCad schematic (older format))
At the start: 0 parts

Commit message: Mostly done with the schematic for the lighting system.
Parts:
- added C?: 1u, symbol C
- added C? (x7): 100n, symbol C
- added C? (x2): 10u, symbol CP
- added P?: CONN_01X09, symbol CONN_01X09
- added P?: CONN_01X02, symbol CONN_01X02
- added R? (x5): 1K, symbol R
- added RV?: 100K, symbol POT
- added U?: Arduino_Pro_Mini, symbol Arduino_Pro_Mini
- added U? (x4): MCP4131, symbol MCP4131
- added U?: Sparkfun_BOB-11420, symbol Sparkfun_BOB-11420
- added U?: Sparkfun_BOB-08688, symbol Sparkfun_BOB-08688
- added U?: R-78E3.3-0.5, symbol R-78E3.3-0.5
Connections:
- new net: C?.1, U?.5 (P0A), U?.5 (P0A), U?.5 (P0A), U?.5 (P0A)
- new net: R?.2, U?.6 (P0W) (x4)
- new net: P?.1 (P1), R?.1
- new net: P?.3 (P3), R?.1
- new net: P?.5 (P5), R?.1
- new net: P?.7 (P7), R?.1
- new net: C?.2, U?.13 (OUT+)
- new net: R?.1, RV?.2
- new net: C?.1, P?.2 (P2), U?.1 (VIN)
- new net AD-1: U?.1 (SIG), U?.17 (A0/D14)
- new net AD-2: R?.2, U?.18 (A1/D15)
- new net CS-1: U?.15 (FSYNC(CS)), U?.5 (D2)
- new net CS-2: U?.1 (~CS), U?.6 (D3)
- new net CS-3: U?.1 (~CS), U?.7 (D4)
- new net CS-4: U?.1 (~CS), U?.8 (D5)
- new net CS-5: U?.1 (~CS), U?.9 (D6)
- new net GND: C?.2, C?.2, C?.2, C?.2, C?.2, C?.2, C?.2, C?.2, C?.2, P?.1 (P1), P?.2 (P2), P?.4 (P4), P?.6 (P6), P?.8 (P8), RV?.1, U?.14 (OUT-), U?.2 (GND), U?.2 (GND), U?.23 (GND), U?.25 (GND), U?.4 (GND), U?.4 (GND), U?.4 (VSS), U?.4 (VSS), U?.4 (VSS), U?.4 (VSS), U?.7 (P0B), U?.7 (P0B), U?.7 (P0B), U?.7 (P0B)
- new net MOSI: U?.14 (D11), U?.16 (SDATA), U?.3 (SDI/SDO), U?.3 (SDI/SDO), U?.3 (SDI/SDO), U?.3 (SDI/SDO)
- new net OUT_EN: U?.13 (D10)
- new net SCLK: U?.16 (D13), U?.18 (SCLK), U?.2 (SCK), U?.2 (SCK), U?.2 (SCK), U?.2 (SCK)
- new net VDD: C?.1, C?.1, C?.1, C?.1, C?.1, C?.1, C?.1, C?.1, RV?.3, U?.21 (VCC), U?.23 (VIN), U?.3 (VCC), U?.3 (VOUT), U?.8 (VDD), U?.8 (VDD), U?.8 (VDD), U?.8 (VDD)
- no-connect marks 0 -> 11
Other:
- note added: "12V to 3V3 Regulator"
- note added: "Amplifier\nConnections"
- note added: "Decoupling Capacitors"
- note added: "Digital Potentiometers"
- note added: "Sine Wave Generator"
- note removed: "Arduino Pro Mini"
- note removed: "Connections to Amplifier"
- note removed: "Digital Pots"
- note removed: "Waveform Generator"

Commit message: More updates and a datasheet.
Parts:
- removed C? (x2): 100n, symbol C
- added R2, R3: 100K, symbol R
- added U9: IRF9952, symbol IRF9952
- C1, C2: renamed from C?; DigiKey (none) -> 732-8625-1-ND; SparkFun (none) -> -
- C3, C4, C5, C6, C7: renamed from C?; DigiKey (none) -> BC2665CT-ND; SparkFun (none) -> -
- R1, R4, R5, R6, R7: renamed from R?; DigiKey (none) -> CF14JT1K00CT-ND; SparkFun (none) -> -
- U1: renamed from U?; DigiKey (none) -> 945-1661-5-ND; SparkFun (none) -> -
- U2: renamed from U?; DigiKey (none) -> -; SparkFun (none) -> DEV-11114
- U3: renamed from U?; DigiKey (none) -> -; SparkFun (none) -> BOB-08688
- U4: renamed from U?; DigiKey (none) -> -; SparkFun (none) -> BOB-11420
- U5, U6, U7, U8: renamed from U?; DigiKey (none) -> -; SparkFun (none) -> COM-10613
- gave numbers to parts that had none: 4
Connections:
- net GND: now also R2.1, U9.1 (S1)
- net OUT_EN: now also R2.2, U9.2 (G1)
- net at P2.9 (P9): now also U9.5 (D2), U9.6 (D2)
- net +12V: now reaches C1.1, P1.2 (P2), U1.1 (VIN)
- net +12V: now also R3.2, U9.3 (S2)
- net VDD renamed +3V3
- new net: R3.1, U9.4 (G2), U9.7 (D1), U9.8 (D1)
